File: PCB/RemoteControl/RemoteControl.kicad_sch (KiCad schematic)
At the start: 10 parts, among them J1 USB_C_Receptacle_USB2.0_14P, J2 Conn_01x05_Socket, J3 Conn_01x05_Pin, J4 Conn_01x04_Socket, U1 STM32L031K6Tx, U2 TC1262-33

Commit message: push
Parts:
- J2: footprint Connector_Phoenix_MC:PhoenixContact_MC_1,5_5-G-3.5_1x05_P3.50mm_Horizontal -> Connector_PinHeader_1.00mm:PinHeader_1x05_P1.00mm_Horizontal
- J3: footprint Connector_Phoenix_MC:PhoenixContact_MCV_1,5_5-G-3.5_1x05_P3.50mm_Vertical -> Connector_PinHeader_1.00mm:PinHeader_1x05_P1.00mm_Vertical
- J4: footprint Connector_Phoenix_MC:PhoenixContact_MC_1,5_4-G-3.5_1x04_P3.50mm_Horizontal -> Connector_PinHeader_1.00mm:PinHeader_1x04_P1.00mm_Horizontal
Changed lines of the file:
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@@
 			)
 		)
-		(property "Footprint" "Connector_Phoenix_MC:PhoenixContact_MC_1,5_5-G-3.5_1x05_P3.50mm_Horizontal"
+		(property "Footprint" "Connector_PinHeader_1.00mm:PinHeader_1x05_P1.00mm_Horizontal"
 			(at 53.34 92.71 0)
 			(effects
@@
 			)
 		)
-		(property "Footprint" "Connector_Phoenix_MC:PhoenixContact_MCV_1,5_5-G-3.5_1x05_P3.50mm_Vertical"
+		(property "Footprint" "Connector_PinHeader_1.00mm:PinHeader_1x05_P1.00mm_Vertical"
 			(at 21.59 25.4 0)
 			(effects
@@
 			)
 		)
-		(property "Footprint" "Connector_Phoenix_MC:PhoenixContact_MC_1,5_4-G-3.5_1x04_P3.50mm_Horizontal"
+		(property "Footprint" "Connector_PinHeader_1.00mm:PinHeader_1x04_P1.00mm_Horizontal"
 			(at 81.28 92.71 0)
 			(effects

Commit message: Passing DRC
Parts:
- added BT1: Battery, Battery:BatteryHolder_MPD_BC2AAPC_2xAA, symbol Device:Battery
- added J5: Conn_01x06_Socket, Connector_PinSocket_1.00mm:PinSocket_1x06_P1.00mm_Vertical_SMD_Pin1Right, symbol Connector:Conn_01x06_Socket
- J2: footprint Connector_PinHeader_1.00mm:PinHeader_1x05_P1.00mm_Horizontal -> Connector_PinSocket_2.00mm:PinSocket_1x05_P2.00mm_Horizontal
- J4: footprint Connector_PinHeader_1.00mm:PinHeader_1x04_P1.00mm_Horizontal -> Connector_PinSocket_2.00mm:PinSocket_1x04_P2.00mm_Horizontal
Connections:
- net +5V: now also BT1.1 (+)
- net GND: now also BT1.2 (-), J5.1 (Pin_1)
- net debug_tx: now reaches U1.19 (PA9)
- net debug_tx: now also J5.4 (Pin_4)
- net debug_rx: now reaches U1.20 (PA10)
- net debug_rx: now also J5.5 (Pin_5)
- no-connect marks 23 -> 24
Other:
- moved on the sheet: C1, C2, D1, J1, J2, J3, J4, R1, U1, U2

Commit message: Pushing
Parts:
- removed J2: Conn_01x05_Socket, Connector_PinSocket_2.00mm:PinSocket_1x05_P2.00mm_Horizontal, symbol Connector:Conn_01x05_Socket
- removed J4: Conn_01x04_Socket, Connector_PinSocket_2.00mm:PinSocket_1x04_P2.00mm_Horizontal, symbol Connector:Conn_01x04_Socket
- added J4, J6, J7, J8, J9: Conn_01x02_Socket, Connector_PinSocket_2.00mm:PinSocket_1x02_P2.00mm_Horizontal, symbol Connector:Conn_01x02_Socket
- added R2, R3, R4, R5, R6: R, Resistor_SMD:R_0805_2012Metric_Pad1.20x1.40mm_HandSolder, symbol Device:R
- added U3: NORA-W106-00B, NORA-W106-00B:XCVR_NORA-W106-00B, symbol NORA-W106-00B:NORA-W106-00B
- J3: footprint Connector_PinHeader_1.00mm:PinHeader_1x05_P1.00mm_Vertical -> Connector_PinHeader_2.00mm:PinHeader_1x05_P2.00mm_Vertical_SMD_Pin1Right
Connections:
- net +3.3V: now also J4.2 (Pin_2), J6.2 (Pin_2), J7.2 (Pin_2), J8.2 (Pin_2), J9.2 (Pin_2), U3.A8 (VCC)
- net Finger1: now also J9.1 (Pin_1), R2.2
- net Finger2: now also J8.1 (Pin_1), R3.2
- net Finger3: now also U1.11 (PA5), J7.1 (Pin_1), R4.2; no longer U1.10 (PA4)
- net Finger4: now also U1.9 (PA3), J6.1 (Pin_1), R5.2; no longer U1.11 (PA5)
- net Finger5: now also U1.8 (PA2), J4.1 (Pin_1), R6.2; no longer U1.12 (PA6)
- net GND: now also R2.1, R3.1, R4.1, R5.1, R6.1, U3.A1 (EGP), U3.A9 (EGP), U3.B2 (EGP), U3.B8 (EGP), U3.E4 (EGP), U3.E5 (EGP), U3.F4 (EGP), U3.F5 (EGP), U3.K2 (EGP), U3.K3 (EGP), U3.K5 (EGP), U3.K7 (EGP), U3.K8 (EGP)
- net RX: now also U1.10 (PA4), U3.G9 (U0RXD/GPIO44); no longer U1.9 (PA3)
- net TX: now also U1.12 (PA6), U3.G8 (U0TXD/GPIO43); no longer U1.8 (PA2)
- net debug_rx: now also U1.19 (PA9); no longer U1.20 (PA10)
- net debug_tx: now also U1.20 (PA10); no longer U1.19 (PA9)
- new net: U3.A4 (NC), U3.B5 (NC), U3.B9 (NC), U3.C5 (NC), U3.D7 (NC), U3.G4 (NC), U3.G5 (NC), U3.G7 (NC), U3.J4 (NC), U3.J5 (NC), U3.J7 (NC), U3.K1 (NC)
- new net: U3.A7 (VCCIO), U3.B7 (VCCIO)
- new net: U3.L1 (EAGP), U3.L9 (EAGP), U3.M1 (EAGP), U3.M2 (EAGP), U3.M8 (EAGP), U3.M9 (EAGP)
- no-connect marks 24 -> 73
