File: PCB/RemoteControl/RemoteControl.kicad_sch (KiCad schematic)
At the start: 24 parts, among them J1 USB_C_Receptacle_USB2.0_14P, J2 Conn_01x02_Pin, J3 Conn_01x05_Pin, J4 Conn_01x02_Socket, J5 Conn_01x06_Socket, J6 Conn_01x02_Socket, J7 Conn_01x02_Socket, J8 Conn_01x02_Socket, J9 Conn_01x02_Socket, U1 STM32L031K6Tx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

Commit message: wasd
Parts:
- added C3, C4, C5, C6, C7: .1u, Capacitor_SMD:C_0504_1310Metric_Pad0.83x1.28mm_HandSolder, symbol Device:C
- added D2: LED, LED_SMD:LED_1206_3216Metric_Pad1.42x1.75mm_HandSolder, symbol Device:LED
- added J10: Conn_01x01_Pin, symbol Connector:Conn_01x01_Pin
- added R8: 270, Resistor_SMD:R_0805_2012Metric_Pad1.20x1.40mm_HandSolder, symbol Device:R
- added R9: R, Resistor_SMD:R_0805_2012Metric_Pad1.20x1.40mm_HandSolder, symbol Device:R
- added TP1, TP3, TP4, TP5, TP6: TestPoint, TestPoint:TestPoint_Pad_2.5x2.5mm, symbol Connector:TestPoint
Connections:
- net +3.3V: now also U3.A7 (VCCIO), U3.B7 (VCCIO), C3.1, C4.1, C5.1, C6.1, C7.1
- net Finger1: now also TP1.1
- net Finger2: now also TP3.1
- net Finger3: now also U1.10 (PA4), TP6.1; no longer U1.8 (PA2)
- net Finger4: now also U1.11 (PA5), TP5.1; no longer U1.9 (PA3)
- net Finger5: now also U1.12 (PA6), TP4.1; no longer U1.11 (PA5)
- net GND: now also C3.2, C4.2, C5.2, C6.2, C7.2, D2.1 (K), R9.1; no longer U1.31 (BOOT0)
- net RX: now also U1.8 (PA2); no longer U1.10 (PA4)
- net TX: now also U1.9 (PA3); no longer U1.12 (PA6)
- net UART_RTS->BoardCTS: now reaches U3.F8 (GPIO45)
- net UART_RTS->BoardCTS: now also U1.21 (PA11)
- net UART_CTS->BoardRTS: now reaches U3.F9 (GPIO6)
- net UART_CTS->BoardRTS: now also U1.14 (PB0)
- net GreenLED: now reaches U3.H8 (GPIO2)
- net GreenLED: now also D4.3 (GK)
- net at U1.15 (PB1): now also R8.1
- new net: D2.2 (A), R8.2
- new net BootPin: J10.1 (Pin_1), R9.2, U1.31 (BOOT0)
- no-connect marks 63 -> 55
