File: PCB/RemoteControl/RemoteControl.kicad_pcb (KiCad board)
At the start: 2 copper layers, 44 x 54.5 mm, 14 parts, among them J1 USB_C_Receptacle_USB2.0_14P, J2 Conn_02x05_Top_Bottom, J3 Conn_01x06, J4 Conn_01x03, SW1 SW_Push, U1 STM32L031K6Tx, U2 TC1262-33

Commit message: push
Parts:
- removed D2: LED, LED_SMD:LED_0805_2012Metric_Pad1.15x1.40mm_HandSolder
- removed R2, R3: 330, Resistor_SMD:R_0805_2012Metric_Pad1.20x1.40mm_HandSolder
- removed SW1: SW_Push, Button_Switch_THT:SW_PUSH_6mm_H4.3mm
- C1: value .1uf -> .1u; footprint Capacitor_SMD:C_0805_2012Metric_Pad1.18x1.45mm_HandSolder -> Capacitor_SMD:C_0504_1310Metric_Pad0.83x1.28mm_HandSolder
- C2: value 10uf -> 1; footprint Capacitor_SMD:C_0805_2012Metric_Pad1.18x1.45mm_HandSolder -> Capacitor_SMD:C_0504_1310Metric_Pad0.83x1.28mm_HandSolder
- D1: footprint LED_SMD:LED_0805_2012Metric_Pad1.15x1.40mm_HandSolder -> LED_SMD:LED_1206_3216Metric_Pad1.42x1.75mm_HandSolder
- J2: value Conn_02x05_Top_Bottom -> Conn_01x05_Socket; footprint Connector_PinHeader_2.54mm:PinHeader_2x05_P2.54mm_Vertical -> Connector_PinHeader_1.00mm:PinHeader_1x05_P1.00mm_Horizontal
- J3: value Conn_01x06 -> Conn_01x05_Pin; footprint Connector_PinHeader_2.54mm:PinHeader_1x06_P2.54mm_Vertical -> Connector_PinHeader_1.00mm:PinHeader_1x05_P1.00mm_Vertical
- J4: value Conn_01x03 -> Conn_01x04_Socket; footprint Connector_PinHeader_2.54mm:PinHeader_1x03_P2.54mm_Vertical -> Connector_PinHeader_1.00mm:PinHeader_1x04_P1.00mm_Horizontal
- R1: value 4.7k -> 270
- moved J1 61.1 mm to (66.3, 25.9), turned to 180 degrees
- moved U2 52.6 mm to (52.0, 25.5), turned to 90 degrees
- moved D1 43.8 mm to (59.5, 32.5), turned to 180 degrees
- moved C2 17.2 mm to (53.9, 39.0), turned to 180 degrees
- moved C1 16.7 mm to (53.9, 36.0), turned to 180 degrees
- moved U1 13.4 mm to (41.5, 30.5), turned to -90 degrees
- moved R1 13.0 mm to (54.0, 32.5), turned to 0 degrees
- moved J3 12.2 mm to (46.5, 37.2), turned to -90 degrees
- moved J2 11.9 mm to (40.0, 40.0), turned to -90 degrees
- moved J4 5.98 mm to (68.5, 31.8)
Connections:
- C1 pad 1: VAPP -> +3.3V
- C2 pad 1: VAPP -> +3.3V
- J2 pad 1: unconnected-(J2-Pin_1-Pad1) -> Finger1
- J2 pad 2: unconnected-(J2-Pin_2-Pad2) -> Finger2
- J2 pad 3: unconnected-(J2-Pin_3-Pad3) -> Finger3
- J2 pad 4: unconnected-(J2-Pin_4-Pad4) -> Finger4
- J2 pad 5: unconnected-(J2-Pin_5-Pad5) -> Finger5
- J3 pad 1: rx -> +3.3V
- J3 pad 2: tx -> GND
- J3 pad 3: GND -> SWSCLK
- J3 pad 4: unconnected-(J3-Pin_4-Pad4) -> SWDIO
- J3 pad 5: unconnected-(J3-Pin_5-Pad5) -> NRST
- J4 pad 1: SDA -> RX
- J4 pad 2: SCL -> TX
- R1 pad 1: NRST -> +3.3V
- R1 pad 2: VAPP -> Net-(D1-A)
- U1 pad 1: VAPP -> +3.3V
- U1 pad 10: unconnected-(U1-PA4-Pad10) -> Finger3
- U1 pad 11: unconnected-(U1-PA5-Pad11) -> Finger4
- U1 pad 12: unconnected-(U1-PA6-Pad12) -> Finger5
- U1 pad 14: Net-(U1-PB0) -> unconnected-(U1-PB0-Pad14)
- U1 pad 17: VAPP -> +3.3V
- U1 pad 19: SCL -> unconnected-(U1-PA9-Pad19)
- U1 pad 20: SDA -> unconnected-(U1-PA10-Pad20)
- U1 pad 23: TMS_SWDIO -> SWDIO
- U1 pad 24: TCK_SWCLK -> SWSCLK
- U1 pad 5: VAPP -> +3.3V
- U1 pad 6: unconnected-(U1-PA0-Pad6) -> Finger1
- U1 pad 7: unconnected-(U1-PA1-Pad7) -> Finger2
- U1 pad 8: tx -> TX
- U1 pad 9: rx -> RX
- U2 pad 3: VAPP -> +3.3V
Routing:
- net GND: track 286.6 -> 16.0 mm
- net VAPP: track 189.8 -> 0.00 mm, vias 3 -> 0
- net TMS_SWDIO: track 79.7 -> 0.00 mm, vias 4 -> 0
- net NRST: track 56.0 -> 0.00 mm, vias 1 -> 0
- net TCK_SWCLK: track 47.8 -> 0.00 mm, vias 2 -> 0
- net Net-(U1-PB0): track 32.1 -> 0.00 mm
- net +5V: track 49.4 -> 18.6 mm
- net RX: track 0.00 -> 30.9 mm
- net Finger2: track 0.00 -> 28.0 mm, vias 0 -> 2
- net rx: track 22.6 -> 0.00 mm
- net Finger1: track 0.00 -> 15.3 mm
- net tx: track 14.4 -> 0.00 mm
- net Finger3: track 0.00 -> 13.0 mm, vias 0 -> 2
- net SDA: track 11.8 -> 0.00 mm, vias 1 -> 0
- net Finger4: track 0.00 -> 11.6 mm, vias 0 -> 2
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- added copper zone on B.Cu, net +3.3V
- removed copper zone on B.Cu, net VAPP
Other:
- board size 44 x 54.5 mm -> 36.8 x 21.8 mm
- board text removed: "gnd"
- board text removed: "rx"
- board text removed: "tx"

Commit message: Passing DRC
Parts:
- added BT1: Battery, Battery:BatteryHolder_MPD_BC2AAPC_2xAA, F.Cu at (116.2, 109.8)
- added J5: Conn_01x06_Socket, Connector_PinSocket_1.00mm:PinSocket_1x06_P1.00mm_Vertical_SMD_Pin1Right, F.Cu at (68.6, 74.2)
- J2: footprint Connector_PinHeader_1.00mm:PinHeader_1x05_P1.00mm_Horizontal -> Connector_PinSocket_2.00mm:PinSocket_1x05_P2.00mm_Horizontal
- J4: footprint Connector_PinHeader_1.00mm:PinHeader_1x04_P1.00mm_Horizontal -> Connector_PinSocket_2.00mm:PinSocket_1x04_P2.00mm_Horizontal
- moved J1 84.8 mm to (93.1, 106.3), turned to 0 degrees
- moved U2 82.6 mm to (98.5, 93.8), turned to 0 degrees
- moved J4 76.0 mm to (72.6, 107.6), turned to 90 degrees
- moved U1 66.6 mm to (89.9, 76.2), turned to 180 degrees
- moved C2 57.9 mm to (60.3, 96.5), turned to 0 degrees
- moved C1 55.8 mm to (60.3, 91.4), turned to 0 degrees
- moved J3 54.5 mm to (68.1, 87.3), turned to 180 degrees
- moved D1 43.8 mm to (61.6, 76.2), turned to 0 degrees
- moved J2 43.7 mm to (80.2, 57.1)
- moved R1 39.4 mm to (62.0, 71.1)
Connections:
- net GND renamed gnd
- U1 pad 19: unconnected-(U1-PA9-Pad19) -> debug_tx
- U1 pad 20: unconnected-(U1-PA10-Pad20) -> debug_rx
Routing:
- net NRST: track 0.00 -> 40.3 mm, vias 0 -> 1
- net Finger2: track 28.0 -> 0.00 mm, vias 2 -> 0
- net +5V: track 18.6 -> 45.1 mm
- net Finger1: track 15.3 -> 0.00 mm
- net Finger3: track 13.0 -> 0.00 mm, vias 2 -> 0
- net Finger4: track 11.6 -> 0.00 mm, vias 2 -> 0
- net Finger5: track 11.4 -> 0.00 mm
- net +3.3V: track 11.1 -> 0.00 mm, vias 1 -> 6
- net RX: track 30.9 -> 20.8 mm, vias 0 -> 1
- net gnd: track 16.0 -> 10.6 mm
- net TX: track 3.50 -> 5.25 mm
- net (no net): vias 0 -> 1
Other:
- board size 36.8 x 21.8 mm -> 86.4 x 56.6 mm

Commit message: Pushing
Parts:
- removed J2: Conn_01x05_Socket, Connector_PinSocket_2.00mm:PinSocket_1x05_P2.00mm_Horizontal
- added J6: Conn_01x02_Socket, Connector_PinSocket_2.00mm:PinSocket_1x02_P2.00mm_Horizontal, F.Cu at (95.0, 119.6)
- added J7: Conn_01x02_Socket, Connector_PinSocket_2.00mm:PinSocket_1x02_P2.00mm_Horizontal, F.Cu at (111.9, 119.7)
- added J8: Conn_01x02_Socket, Connector_PinSocket_2.00mm:PinSocket_1x02_P2.00mm_Horizontal, F.Cu at (128.9, 119.9)
- added J9: Conn_01x02_Socket, Connector_PinSocket_2.00mm:PinSocket_1x02_P2.00mm_Horizontal, F.Cu at (146.4, 120.3)
- added R2: R, Resistor_SMD:R_0805_2012Metric_Pad1.20x1.40mm_HandSolder, F.Cu at (146.4, 113.4)
- added R3: R, Resistor_SMD:R_0805_2012Metric_Pad1.20x1.40mm_HandSolder, F.Cu at (128.9, 113.1)
- added R4: R, Resistor_SMD:R_0805_2012Metric_Pad1.20x1.40mm_HandSolder, F.Cu at (111.9, 113.2)
- added R5: R, Resistor_SMD:R_0805_2012Metric_Pad1.20x1.40mm_HandSolder, F.Cu at (95.1, 113.0)
- added R6: R, Resistor_SMD:R_0805_2012Metric_Pad1.20x1.40mm_HandSolder, F.Cu at (79.1, 113.0)
- added U3: NORA-W106-00B, NORA-W106-00B:XCVR_NORA-W106-00B, F.Cu at (76.3, 58.3)
- J3: footprint Connector_PinHeader_1.00mm:PinHeader_1x05_P1.00mm_Vertical -> Connector_PinHeader_2.00mm:PinHeader_1x05_P2.00mm_Vertical_SMD_Pin1Right
- J4: value Conn_01x04_Socket -> Conn_01x02_Socket; footprint Connector_PinSocket_2.00mm:PinSocket_1x04_P2.00mm_Horizontal -> Connector_PinSocket_2.00mm:PinSocket_1x02_P2.00mm_Horizontal
- moved BT1 72.5 mm to (162.7, 54.2), turned to -90 degrees
- moved C2 72.1 mm to (127.7, 70.9), turned to 180 degrees
- moved J5 64.6 mm to (130.4, 93.2)
- moved J1 55.5 mm to (112.9, 54.5), turned to 180 degrees
- moved C1 43.3 mm to (103.2, 85.2)
- moved U2 41.2 mm to (126.5, 63.6), turned to 90 degrees
- moved D1 35.7 mm to (97.3, 78.3), turned to 180 degrees
- moved R1 26.7 mm to (87.7, 78.3)
- moved U1 26.1 mm to (108.6, 94.5), turned to 0 degrees
- moved J3 14.0 mm to (80.6, 93.6), turned to 0 degrees
- moved J4 13.3 mm to (79.0, 119.3)
Connections:
- J4 pad 1: RX -> Finger5
- J4 pad 2: TX -> +3.3V
- U1 pad 10: Finger3 -> RX
- U1 pad 11: Finger4 -> Finger3
- U1 pad 12: Finger5 -> TX
- U1 pad 19: debug_tx -> debug_rx
- U1 pad 20: debug_rx -> debug_tx
- U1 pad 8: TX -> Finger5
- U1 pad 9: RX -> Finger4
Routing:
- net +3.3V: track 0.00 -> 89.9 mm, vias 6 -> 8
- net TX: track 5.25 -> 90.5 mm, vias 1 -> 2
- net Finger1: track 0.00 -> 73.8 mm, vias 0 -> 2
- net RX: track 20.8 -> 82.1 mm, vias 1 -> 2
- net Finger2: track 0.00 -> 54.4 mm, vias 0 -> 2
- net SWDIO: track 0.00 -> 54.1 mm
- net SWSCLK: track 0.00 -> 50.9 mm, vias 0 -> 2
- net gnd: track 10.6 -> 52.5 mm
- net Finger5: track 0.00 -> 41.0 mm
- net debug_rx: track 0.00 -> 33.6 mm
- net +5V: track 45.1 -> 74.3 mm
- net Finger4: track 0.00 -> 25.4 mm
- net Finger3: track 0.00 -> 23.0 mm
- net debug_tx: track 0.00 -> 17.9 mm
- net NRST: track 40.3 -> 26.0 mm, vias 1 -> 0
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Other:
- board size 86.4 x 56.6 mm -> 106.8 x 80.3 mm

Commit message: Stuff
Routing:
- net +5V: track 74.3 -> 72.3 mm
- net gnd: track 52.5 -> 50.7 mm, vias 0 -> 4
- net debug_tx: track 17.9 -> 17.1 mm
Changed lines of the file:
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@@
-	)
-	(segment
-		(start 120.269 57.9882)
-		(end 120.269 66.6496)
-		(width 0.2)
-		(layer "F.Cu")
-		(net 6)
-	)
-	(segment
-		(start 120.1928 66.7766)
-		(end 124.1806 66.7766)
-		(width 0.2)
-		(layer "F.Cu")
-		(net 6)
 	)
 	(segment
@@
 	)
 	(segment
-		(start 120.269 66.6496)
-		(end 120.1674 66.7512)
+		(start 115.453546 57.9882)
+		(end 118.8 57.9882)
+		(width 0.2)
+		(layer "F.Cu")
+		(net 6)
+	)
+	(segment
+		(start 124.1806 66.7766)
+		(end 124.1806 63.3688)
 		(width 0.2)
 		(layer "F.Cu")
@@
 	)
 	(segment
-		(start 120.4468 57.9882)
-		(end 120.269 57.9882)
-		(width 0.2)
-		(layer "F.Cu")
-		(net 6)
-	)
-	(segment
 		(start 107.8062 54.590854)
 		(end 108.386546 55.1712)
@@
 	)
 	(segment
-		(start 115.453546 57.9882)
+		(start 118.8 57.9882)
 		(end 120.4468 57.9882)
 		(width 0.2)
@@
 	)
 	(segment
-		(start 120.1674 66.7512)
-		(end 120.1928 66.7766)
+		(start 124.1806 63.3688)
+		(end 118.8 57.9882)
 		(width 0.2)
 		(layer "F.Cu")
@@
 	)
 	(segment
-		(start 122.2596 93.7354)
-		(end 122.1486 93.6244)
-		(width 0.2)
-		(layer "F.Cu")
-		(net 23)
-	)
-	(segment
-		(start 122.174 94.7928)
-		(end 122.1136 94.8532)
+		(start 123.2314 93.7354)
+		(end 129.3934 93.7354)
 		(width 0.2)
 		(layer "F.Cu")
@@
 	)
 	(segment
-		(start 129.3934 93.7354)
-		(end 122.2596 93.7354)
+		(start 122.1136 94.8532)
+		(end 123.2314 93.7354)
 		(width 0.2)
 		(layer "F.Cu")
@@
 	)
 	(segment
-		(start 122.1486 93.6244)
-		(end 122.1486 94.7674)
-		(width 0.2)
-		(layer "F.Cu")
-		(net 23)
-	)
-	(segment
-		(start 122.1486 94.7674)
-		(end 122.174 94.7928)
-		(width 0.2)
-		(layer "F.Cu")
-		(net 23)
-	)
-	(segment
-		(start 92.9132 97.663)
+		(start 92.9264 97.6498)
 		(end 93.1672 97.409)
 		(width 0.2)
@@
 	)
 	(segment
+		(start 93.3226 94.0532)
+		(end 104.3782 94.0532)
+		(width 0.2)
+		(layer "F.Cu")
+		(net 31)
+	)
+	(segment
+		(start 93.1672 94.2086)
+		(end 93.3226 94.0532)
+		(width 0.2)
+		(layer "F.Cu")
+		(net 31)
+	)
+	(segment
 		(start 81.7372 97.6498)
-		(end 92.9 97.6498)
-		(width 0.2)
-		(layer "F.Cu")
-		(net 31)
-	)
-	(segment
-		(start 93.1672 94.2086)
-		(end 93.345 94.2086)
-		(width 0.2)
-		(layer "F.Cu")
-		(net 31)
-	)
-	(segment
-		(start 93.5004 94.0532)
-		(end 104.3782 94.0532)
-		(width 0.2)
-		(layer "F.Cu")
-		(net 31)
-	)
-	(segment
-		(start 92.9 97.6498)
-		(end 92.9132 97.663)
-		(width 0.2)
-		(layer "F.Cu")
-		(net 31)
-	)
-	(segment
-		(start 93.345 94.2086)
-		(end 93.5004 94.0532)
+		(end 92.9264 97.6498)
 		(width 0.2)
 		(layer "F.Cu")
@@
 	)
 	(segment
-		(start 76.8096 60.2898)
-		(end 76.8096 59.1898)
-		(width 0.2)
-		(layer "F.Cu")
-		(net 43)
-	)
-	(segment
 		(start 71.8596 64.6898)
 		(end 72.9596 63.5898)
@@
 	)
 	(segment
-		(start 76.0984 59.2582)
-		(end 76.03 59.1898)
-		(width 0.2)
-		(layer "F.Cu")
-		(net 43)
-	)
-	(segment
-		(start 75.7096 59.1898)
-		(end 75.7096 60.2898)
-		(width 0.2)
-		(layer "F.Cu")
-		(net 43)
-	)
-	(segment
 		(start 72.9596 54.7898)
 		(end 79.5596 54.7898)
@@
 	)
 	(segment
-		(start 75.7096 60.2898)
-		(end 75.7096 60.8398)
-		(width 0.2)
-		(layer "F.Cu")
-		(net 43)
-	)
-	(segment
 		(start 79.5596 63.5898)
 		(end 79.5596 63.4814)
@@
 	)
 	(segment
-		(start 76.03 59.1898)
-		(end 75.7096 59.1898)
-		(width 0.2)
-		(layer "F.Cu")
-		(net 43)
-	)
-	(segment
-		(start 75.7096 60.8398)
-		(end 72.9596 63.5898)
-		(width 0.2)
-		(layer "F.Cu")
-		(net 43)
-	)
-	(segment
-		(start 76.1668 59.1898)
-		(end 76.0984 59.2582)
-		(width 0.2)
-		(layer "F.Cu")
-		(net 43)
-	)
-	(segment
-		(start 75.7096 60.2898)
-		(end 76.8096 60.2898)
-		(width 0.2)
-		(layer "F.Cu")
-		(net 43)
-	)
-	(segment
 		(start 76.8096 60.8398)
 		(end 79.5596 63.5898)
@@
 		(net 43)
 	)
-	(segment
-		(start 79.5596 63.4814)
-		(end 79.169 63.0908)
-		(width 0.2)
-		(layer "F.Cu")
-		(net 43)
-	)
-	(segment
-		(start 76.8096 59.1898)
-		(end 76.1668 59.1898)
-		(width 0.2)
-		(layer "F.Cu")
-		(net 43)
-	)
+	(via
+		(at 95.8 85.5)
+		(size 0.6)
+		(drill 0.3)
+		(layers "F.Cu" "B.Cu")
+		(net 43)
+	)
+	(via
+		(at 125.7 88.1)
+		(size 0.6)
+		(drill 0.3)
+		(layers "F.Cu" "B.Cu")
+		(free yes)
+		(net 43)
+	)
+	(via
+		(at 125.7 84.4)
+		(size 0.6)
+		(drill 0.3)
+		(layers "F.Cu" "B.Cu")
+		(net 43)
+	)
+	(via
+		(at 95.8 89.5)
+		(size 0.6)
+		(drill 0.3)
+		(layers "F.Cu" "B.Cu")
+		(free yes)
+		(net 43)
+	)
+	(segment
+		(start 95.8 89.5)
+		(end 95.8 85.5)
+		(width 0.2)
+		(layer "B.Cu")
+		(net 43)
+	)
+	(segment
+		(start 125.7 88.1)
+		(end 125.7 84.4)
+		(width 0.2)
+		(layer "B.Cu")
+		(net 43)
+	)

Commit message: Remote Control
Parts:
- removed BT1: Battery, Battery:BatteryHolder_MPD_BC2AAPC_2xAA
- added D4: ASMB-MTB0-0A3A2, LED_SMD:LED_Avago_PLCC4_3.2x2.8mm_CW, F.Cu at (76.4, 54.7)
- added J2: Conn_01x02_Pin, Connector_PinHeader_2.54mm:PinHeader_1x02_P2.54mm_Horizontal, F.Cu at (158.9, 59.2)
- added R7: R, Resistor_SMD:R_0805_2012Metric_Pad1.20x1.40mm_HandSolder, F.Cu at (77.9, 63.1)
- added TP2: TestPoint, TestPoint:TestPoint_Pad_2.5x2.5mm, F.Cu at (90.7, 71.8)
- J3: footprint Connector_PinHeader_2.00mm:PinHeader_1x05_P2.00mm_Vertical_SMD_Pin1Right -> Connector_PinHeader_2.54mm:PinHeader_1x05_P2.54mm_Vertical
- J4, J6, J7, J8, J9: footprint Connector_PinSocket_2.00mm:PinSocket_1x02_P2.00mm_Horizontal -> Connector_PinSocket_2.54mm:PinSocket_1x02_P2.54mm_Horizontal
- J5: footprint Connector_PinSocket_1.00mm:PinSocket_1x06_P1.00mm_Vertical_SMD_Pin1Right -> Connector_PinHeader_2.54mm:PinHeader_1x06_P2.54mm_Vertical
- moved J3 86.3 mm to (165.2, 76.8)
- moved J9 70.0 mm to (76.4, 117.7)
- moved R2 69.9 mm to (76.6, 108.1)
- moved R4 43.8 mm to (155.4, 108.1)
- moved J7 43.6 mm to (155.4, 117.9)
- moved J6 41.5 mm to (136.5, 118.0)
- moved R5 41.5 mm to (136.3, 108.1)
- moved R1 38.7 mm to (117.5, 53.5), turned to -90 degrees
- moved R6 36.3 mm to (115.1, 108.4)
- moved J4 36.0 mm to (114.9, 117.7)
- moved J5 34.9 mm to (165.3, 92.7)
- moved R3 34.0 mm to (95.2, 108.3)
- moved J8 33.9 mm to (95.1, 117.9)
- moved J1 31.2 mm to (144.1, 54.5)
- moved D1 28.0 mm to (117.4, 58.9), turned to 90 degrees
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Connections:
- net debug_rx renamed debuging_rx
- net debug_tx renamed debuging_tx
- J4 pad 1: Finger5 -> Finger3
- J7 pad 1: Finger3 -> Finger5
- R4 pad 2: Finger3 -> Finger5
- R6 pad 2: Finger5 -> Finger3
- U1 pad 11: Finger3 -> Finger5
- U1 pad 13: unconnected-(U1-PA7-Pad13) -> Net-(U1-PA7)
- U1 pad 26: unconnected-(U1-PB3-Pad26) -> GPIO_J9
- U1 pad 27: unconnected-(U1-PB4-Pad27) -> Switch1
- U1 pad 28: unconnected-(U1-PB5-Pad28) -> Switch2
- U1 pad 8: Finger5 -> Finger3
- U3 pad A5: unconnected-(U3-FSPIDQS/GPIO14-PadA5) -> DEBUG_TX
- U3 pad C8: unconnected-(U3-GPIO21-PadC8) -> Switch2
- U3 pad D8: unconnected-(U3-GPIO4-PadD8) -> Switch1
- U3 pad H9: unconnected-(U3-GPIO8-PadH9) -> BlueLED
- U3 pad J3: unconnected-(U3-~{RESET}-PadJ3) -> Net-(U1-PA7)
- U3 pad J8: unconnected-(U3-GPIO5-PadJ8) -> RedLED
- U3 pad J9: unconnected-(U3-GPIO3-PadJ9) -> GPIO_J9
Routing:
- net GPIO_J9: track 0.00 -> 73.4 mm, vias 0 -> 2
- net +5V: track 72.3 -> 16.9 mm
- net Switch1: track 0.00 -> 49.1 mm, vias 0 -> 2
- net Net-(U1-PA7): track 0.00 -> 49.0 mm, vias 0 -> 2
- net Switch2: track 0.00 -> 47.1 mm, vias 0 -> 2
- net TX: track 90.5 -> 50.4 mm
- net NRST: track 26.0 -> 63.1 mm, vias 0 -> 2
- net +3.3V: track 89.9 -> 55.3 mm, vias 8 -> 11
- net RX: track 82.1 -> 49.9 mm
- net gnd: track 50.7 -> 81.3 mm
- net debuging_tx: track 17.1 -> 43.0 mm
- net BlueLED: track 0.00 -> 22.2 mm
- net SWDIO: track 54.1 -> 37.4 mm
- net SWSCLK: track 50.9 -> 37.1 mm, vias 2 -> 0
- net Finger1: track 73.8 -> 61.5 mm, vias 2 -> 0
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
Commit message: Updated remote control
Parts:
- removed J4, J6: Conn_01x02_Socket, Connector_PinSocket_2.54mm:PinSocket_1x02_P2.54mm_Horizontal
- removed R2, R3: R, Resistor_SMD:R_0805_2012Metric_Pad1.20x1.40mm_HandSolder
- added J10: Conn_01x02_Socket, Connector_PinSocket_2.54mm:PinSocket_1x02_P2.54mm_Horizontal, F.Cu at (123.8, 102.5)
- added J11: Conn_01x02_Socket, Connector_PinSocket_2.54mm:PinSocket_1x02_P2.54mm_Horizontal, F.Cu at (136.6, 102.5)
- added R8: R, Resistor_SMD:R_0805_2012Metric_Pad1.20x1.40mm_HandSolder, F.Cu at (124.8, 96.4)
- added R9: R, Resistor_SMD:R_0805_2012Metric_Pad1.20x1.40mm_HandSolder, F.Cu at (137.6, 96.4)
- moved R5 38.7 mm to (99.5, 96.4), turned to 180 degrees
- moved J9 37.9 mm to (111.2, 102.5)
- moved D4 37.8 mm to (114.2, 54.7)
- moved TP2 37.8 mm to (128.5, 71.8)
- moved R7 37.8 mm to (115.7, 63.1)
- moved U3 37.8 mm to (128.4, 55.9)
- moved D1 32.8 mm to (145.0, 76.8), turned to 180 degrees
- moved R1 32.1 mm to (139.6, 76.7), turned to 0 degrees
- moved J1 18.1 mm to (162.2, 54.5)
- moved J7 16.6 mm to (149.2, 102.5)
- moved J8 15.7 mm to (98.5, 102.5)
- moved C2 14.2 mm to (143.9, 56.2), turned to 0 degrees
- moved R4 12.7 mm to (150.2, 96.4), turned to 180 degrees
- moved R6 12.4 mm to (112.2, 96.4), turned to 180 degrees
- moved J2 6.34 mm to (159.9, 65.5), turned to 0 degrees
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Connections:
- J8 pad 1: Finger2 -> Finger1
- J9 pad 1: Finger1 -> Finger2
- R5 pad 2: Finger4 -> Finger1
- R6 pad 2: Finger3 -> Finger2
Routing:
- net gnd: track 81.3 -> 32.4 mm, vias 4 -> 0
- net GPIO_J9: track 73.4 -> 41.4 mm
- net Finger1: track 61.5 -> 31.8 mm
- net Switch1: track 49.1 -> 22.6 mm
- net Switch2: track 47.1 -> 23.3 mm
- net Finger2: track 42.6 -> 19.4 mm
- net TX: track 50.4 -> 34.2 mm
- net Finger3: track 31.8 -> 16.1 mm
- net RX: track 49.9 -> 34.4 mm
- net Finger5: track 49.8 -> 35.7 mm
- net Finger4: track 34.9 -> 24.8 mm
- net Net-(U1-PA7): track 49.0 -> 40.3 mm
- net NRST: track 63.1 -> 54.3 mm, vias 2 -> 0
- net BlueLED: track 22.2 -> 14.7 mm
- net +5V: track 16.9 -> 22.1 mm
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Other:
- board size 106.8 x 80.3 mm -> 78 x 64.6 mm

Commit message: mwasd
Parts:
- removed J10, J11: Conn_01x02_Socket, Connector_PinSocket_2.54mm:PinSocket_1x02_P2.54mm_Horizontal
- removed R9: R, Resistor_SMD:R_0805_2012Metric_Pad1.20x1.40mm_HandSolder
- added C3: .1u, Capacitor_SMD:C_0504_1310Metric_Pad0.83x1.28mm_HandSolder, F.Cu at (120.7, 62.2)
- added C4: .1u, Capacitor_SMD:C_0504_1310Metric_Pad0.83x1.28mm_HandSolder, F.Cu at (120.6, 64.8)
- added C5: .1u, Capacitor_SMD:C_0504_1310Metric_Pad0.83x1.28mm_HandSolder, F.Cu at (120.6, 59.8)
- added C6: .1u, Capacitor_SMD:C_0504_1310Metric_Pad0.83x1.28mm_HandSolder, F.Cu at (133.4, 88.0)
- added C7: .1u, Capacitor_SMD:C_0504_1310Metric_Pad0.83x1.28mm_HandSolder, F.Cu at (115.2, 84.0)
- added D2: LED, LED_SMD:LED_1206_3216Metric_Pad1.42x1.75mm_HandSolder, F.Cu at (147.4, 92.4)
- added J4: Conn_01x02_Socket, Connector_PinSocket_2.54mm:PinSocket_1x02_P2.54mm_Horizontal, F.Cu at (124.2, 102.3)
- added J6: Conn_01x02_Socket, Connector_PinSocket_2.54mm:PinSocket_1x02_P2.54mm_Horizontal, F.Cu at (135.5, 102.5)
- added R2: R, Resistor_SMD:R_0805_2012Metric_Pad1.20x1.40mm_HandSolder, F.Cu at (103.0, 98.6)
- added R3: R, Resistor_SMD:R_0805_2012Metric_Pad1.20x1.40mm_HandSolder, F.Cu at (112.2, 98.2)
- R8: value R -> 270
- moved R5 37.0 mm to (136.4, 98.2)
- moved R8 16.6 mm to (141.0, 92.4), turned to 0 degrees
- moved R6 13.2 mm to (125.2, 98.0)
- moved J9 13.0 mm to (98.2, 102.3)
- moved J8 12.5 mm to (111.0, 102.5)
- moved TP2 6.84 mm to (132.1, 66.0)
Connections:
- D4 pad 3: unconnected-(D4-GK-Pad3) -> GreenLED
- J8 pad 1: Finger1 -> Finger2
- J9 pad 1: Finger2 -> Finger1
- R5 pad 2: Finger1 -> Finger4
- R6 pad 2: Finger2 -> Finger3
- R8 pad 1: gnd -> HeartBeat
- R8 pad 2: Finger3 -> Net-(D2-A)
- U1 pad 10: RX -> Finger3
- U1 pad 11: Finger5 -> Finger4
- U1 pad 12: TX -> Finger5
- U1 pad 14: unconnected-(U1-PB0-Pad14) -> UART_CTS->BOARD_RTS
- U1 pad 15: unconnected-(U1-PB1-Pad15) -> HeartBeat
- U1 pad 21: unconnected-(U1-PA11-Pad21) -> UART_RTS->BOARD_CTS
- U1 pad 8: Finger3 -> RX
- U1 pad 9: Finger4 -> TX
- U3 pad A7: unconnected-(U3-VCCIO-PadA7)_1 -> +3.3V
- U3 pad B7: unconnected-(U3-VCCIO-PadA7) -> +3.3V
- U3 pad F8: unconnected-(U3-GPIO45-PadF8) -> UART_RTS->BOARD_CTS
- U3 pad F9: unconnected-(U3-GPIO6-PadF9) -> UART_CTS->BOARD_RTS
- U3 pad H8: unconnected-(U3-GPIO2-PadH8) -> GreenLED
Routing:
- net UART_CTS->BOARD_RTS: track 0.00 -> 55.4 mm, vias 0 -> 4
- net UART_RTS->BOARD_CTS: track 0.00 -> 42.1 mm, vias 0 -> 4
- net GreenLED: track 0.00 -> 27.1 mm, vias 0 -> 2
- net NRST: track 54.3 -> 74.3 mm, vias 0 -> 2
- net HeartBeat: track 0.00 -> 16.2 mm
- net +3.3V: track 54.0 -> 67.7 mm, vias 7 -> 8
- net GPIO_J9: track 41.4 -> 51.2 mm
- net gnd: track 32.4 -> 25.5 mm, vias 0 -> 2
- net DEBUG_TX: track 9.58 -> 5.28 mm
- net Net-(D2-A): track 0.00 -> 3.91 mm
- net Switch2: track 23.3 -> 25.8 mm
- net Finger4: track 24.8 -> 22.3 mm
- net Finger3: track 16.1 -> 13.9 mm
- net Finger2: track 19.4 -> 20.7 mm
- net TX: track 34.2 -> 35.2 mm
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Other:
- board text added: "3.3v"
- board text added: "Debug_TX"
- board text added: "gnd"
- board text added: "nrst"
- board text added: "rx"
- board text added: "swdio"
- board text added: "swsclk"
- board text added: "tx"
