File: PCB/RemoteControl/RemoteControl.kicad_pcb (KiCad board)
At the start: 2 copper layers, 78 x 64.6 mm, 31 parts, among them J1 USB_C_Receptacle_USB2.0_14P, J2 Conn_01x02_Pin, J3 Conn_01x05_Pin, J4 Conn_01x02_Socket, J5 Conn_01x06_Socket, J6 Conn_01x02_Socket, J7 Conn_01x02_Socket, J8 Conn_01x02_Socket, J9 Conn_01x02_Socket, U1 STM32L031K6Tx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

Commit message: wasd
Parts:
- added J10: Conn_01x01_Pin, Connector_PinHeader_2.54mm:PinHeader_1x01_P2.54mm_Vertical, F.Cu at (114.4, 72.6)
- added R9: R, Resistor_SMD:R_0805_2012Metric_Pad1.20x1.40mm_HandSolder, F.Cu at (119.5, 71.5)
- added TP1: TestPoint, TestPoint:TestPoint_Pad_2.5x2.5mm, F.Cu at (105.9, 102.1)
- added TP3: TestPoint, TestPoint:TestPoint_Pad_2.5x2.5mm, F.Cu at (118.7, 102.4)
- added TP4: TestPoint, TestPoint:TestPoint_Pad_2.5x2.5mm, F.Cu at (158.0, 102.6)
- added TP5: TestPoint, TestPoint:TestPoint_Pad_2.5x2.5mm, F.Cu at (143.7, 102.3)
- added TP6: TestPoint, TestPoint:TestPoint_Pad_2.5x2.5mm, F.Cu at (131.2, 102.2)
- moved C3 2.72 mm to (120.7, 65.0)
- moved C1 2.57 mm to (114.8, 78.4)
- moved C4 2.43 mm to (120.7, 62.3)
- moved C7 2.01 mm to (113.2, 84.1)
- moved C6 1.48 mm to (134.9, 87.9)
- moved R8 0.23 mm to (141.2, 92.5)
- moved D2 0.10 mm to (147.3, 92.5)
- moved C5 0.07 mm to (120.7, 59.7)
Connections:
- net HeartBeat renamed Net-(U1-PB1)
- net UART_CTS->BOARD_RTS renamed UART_CTS->BoardRTS
- net UART_RTS->BOARD_CTS renamed UART_RTS->BoardCTS
- U1 pad 31: gnd -> BootPin
Routing:
- net BootPin: track 0.00 -> 17.4 mm, vias 0 -> 1
- net Finger5: track 36.5 -> 47.8 mm
- net Finger4: track 22.3 -> 32.3 mm
- net gnd: track 25.5 -> 16.0 mm, vias 2 -> 0
- net Finger2: track 20.7 -> 29.9 mm
- net NRST: track 74.3 -> 65.2 mm, vias 2 -> 4
- net Finger3: track 13.9 -> 22.5 mm
- net RX: track 34.0 -> 41.8 mm
- net UART_CTS->BoardRTS: track 55.4 -> 62.1 mm, vias 4 -> 6
- net Finger1: track 31.8 -> 37.2 mm
- net TX: track 35.2 -> 39.7 mm
- net +3.3V: track 67.7 -> 64.7 mm, vias 8 -> 9
Other:
- outline, holes or cut-outs redrawn
- board text added: "Boot"
