File: PCB/RemoteControl/RemoteControl.kicad_pcb (KiCad board)
At the start: 2 copper layers, 78 x 64.6 mm, 38 parts, among them J1 USB_C_Receptacle_USB2.0_14P, J10 Conn_01x01_Pin, J2 Conn_01x02_Pin, J3 Conn_01x05_Pin, J4 Conn_01x02_Socket, J5 Conn_01x06_Socket, J6 Conn_01x02_Socket, J7 Conn_01x02_Socket, J8 Conn_01x02_Socket, J9 Conn_01x02_Socket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

Commit message: final boards
Parts:
- removed J2: Conn_01x02_Pin, Connector_PinHeader_2.54mm:PinHeader_1x02_P2.54mm_Horizontal
- added J11: Conn_01x02_Socket, Connector_PinSocket_2.54mm:PinSocket_1x02_P2.54mm_Horizontal, F.Cu at (108.5, 84.2)
- added R10: R, Resistor_SMD:R_0805_2012Metric_Pad1.20x1.40mm_HandSolder, F.Cu at (127.7, 110.0)
- added R11: R, Resistor_SMD:R_0805_2012Metric_Pad1.20x1.40mm_HandSolder, F.Cu at (129.2, 125.7)
- added R12: R, Resistor_SMD:R_0805_2012Metric_Pad1.20x1.40mm_HandSolder, F.Cu at (142.2, 109.9)
- added R13: R, Resistor_SMD:R_0805_2012Metric_Pad1.20x1.40mm_HandSolder, F.Cu at (142.9, 125.5)
- added R14: R, Resistor_SMD:R_0805_2012Metric_Pad1.20x1.40mm_HandSolder, F.Cu at (156.8, 125.5)
- added R15: R, Resistor_SMD:R_0805_2012Metric_Pad1.20x1.40mm_HandSolder, F.Cu at (155.6, 110.2)
- added R16: R, Resistor_SMD:R_0805_2012Metric_Pad1.20x1.40mm_HandSolder, F.Cu at (114.5, 109.9)
- added R17: R, Resistor_SMD:R_0805_2012Metric_Pad1.20x1.40mm_HandSolder, F.Cu at (116.8, 125.6)
- added R18: R, Resistor_SMD:R_0805_2012Metric_Pad1.20x1.40mm_HandSolder, F.Cu at (101.2, 109.7)
- added R19: R, Resistor_SMD:R_0805_2012Metric_Pad1.20x1.40mm_HandSolder, F.Cu at (101.2, 125.9)
- added TP10: TestPoint, TestPoint:TestPoint_Pad_2.5x2.5mm, F.Cu at (148.3, 109.8)
- added TP11: TestPoint, TestPoint:TestPoint_Pad_2.5x2.5mm, F.Cu at (134.5, 109.4)
- added TP7: TestPoint, TestPoint:TestPoint_Pad_2.5x2.5mm, F.Cu at (107.4, 109.3)
- added TP8: TestPoint, TestPoint:TestPoint_Pad_2.5x2.5mm, F.Cu at (121.2, 109.3)
- added TP9: TestPoint, TestPoint:TestPoint_Pad_2.5x2.5mm, F.Cu at (162.2, 109.6)
- added U4: LM358APE4, lm358:P8, F.Cu at (138.3, 122.3)
- added U5: LM358APE4, lm358:P8, F.Cu at (152.0, 122.2)
- added U6: LM358APE4, lm358:P8, F.Cu at (166.1, 122.1)
- added U7: LM358APE4, lm358:P8, F.Cu at (125.2, 122.0)
- added U8: LM358APE4, lm358:P8, F.Cu at (111.3, 122.0)
- J1: value USB_C_Receptacle_USB2.0_14P -> Barrel_Jack; footprint Connector_USB:USB_C_Receptacle_GCT_USB4085 -> Connector_BarrelJack:BarrelJack_Wuerth_694106106102_2.0x5.5mm
- moved J1 58.3 mm to (104.0, 57.9)
- moved C2 54.2 mm to (112.3, 100.3), turned to -90 degrees
- moved U2 51.9 mm to (104.1, 96.5), turned to 90 degrees
- moved R4 44.1 mm to (156.7, 140.1), turned to 90 degrees
- moved R6 42.3 mm to (131.6, 139.8), turned to 90 degrees
- moved R5 42.1 mm to (143.5, 139.7), turned to 90 degrees
- moved R3 42.0 mm to (118.7, 139.7), turned to 90 degrees
- moved R2 41.0 mm to (104.1, 139.6), turned to 90 degrees
- moved J5 39.9 mm to (150.6, 55.6), turned to -90 degrees
- moved J6 32.0 mm to (148.4, 131.8)
- moved J4 31.7 mm to (136.2, 131.7)
- moved J8 31.7 mm to (123.0, 131.9)
- moved J7 31.7 mm to (161.3, 131.9)
- moved J9 31.7 mm to (110.2, 131.7)
- moved TP6 29.7 mm to (131.4, 131.9)
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Connections:
- J4 pad 1: Finger3 -> Sensor1
- J6 pad 1: Finger4 -> Sensor2
- J7 pad 1: Finger5 -> Sensor3
- J8 pad 1: Finger2 -> Sensor4
- J9 pad 1: Finger1 -> Sensor5
- R2 pad 2: Finger1 -> Sensor5
- R3 pad 2: Finger2 -> Sensor4
- R4 pad 2: Finger5 -> Sensor3
- R5 pad 2: Finger4 -> Sensor2
- R6 pad 2: Finger3 -> Sensor1
- R7 pad 1: gnd -> +3.3V
- TP1 pad 1: Finger1 -> Sensor5
- TP3 pad 1: Finger2 -> Sensor4
- TP4 pad 1: Finger5 -> Sensor3
- TP5 pad 1: Finger4 -> Sensor2
- TP6 pad 1: Finger3 -> Sensor1
- U3 pad L1: unconnected-(U3-EAGP-PadL1) -> gnd
- U3 pad L9: unconnected-(U3-EAGP-PadL1)_4 -> gnd
- U3 pad M1: unconnected-(U3-EAGP-PadL1)_1 -> gnd
- U3 pad M2: unconnected-(U3-EAGP-PadL1)_2 -> gnd
- U3 pad M8: unconnected-(U3-EAGP-PadL1)_5 -> gnd
- U3 pad M9: unconnected-(U3-EAGP-PadL1)_3 -> gnd
Routing:
- net Sensor5: track 0.00 -> 27.9 mm
- net Sensor1: track 0.00 -> 26.1 mm
- net Sensor2: track 0.00 -> 26.0 mm
- net Sensor4: track 0.00 -> 25.7 mm
- net Sensor3: track 0.00 -> 25.2 mm
- net SWDIO: track 37.4 -> 59.7 mm
- net +3.3V: track 64.7 -> 86.3 mm, vias 9 -> 13
- net Net-(U8-1OUT): track 0.00 -> 21.4 mm
- net SWSCLK: track 37.1 -> 57.8 mm
- net Net-(U6-1OUT): track 0.00 -> 20.5 mm
- net Net-(U4-1OUT): track 0.00 -> 20.4 mm
- net Net-(U5-1OUT): track 0.00 -> 20.2 mm
- net Finger4: track 32.3 -> 52.4 mm
- net Net-(U7-1OUT): track 0.00 -> 19.7 mm
- net Net-(U8-1IN-): track 0.00 -> 18.1 mm
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- added copper zone on B.Cu, net +5V
Other:
- board size 78 x 64.6 mm -> 74.8 x 96.4 mm
- board text added: "4.5V"
- board text added: "f1"
- board text added: "f2"
- board text added: "f3"
- board text added: "f4"
- board text added: "f5"
- board text added: "in1"
- board text added: "in2"
- board text added: "in3"
- board text added: "in4"
- board text added: "in5"
- board text added: "stm_rx"
- board text added: "stm_tx"
- board text removed: "Debug_TX"
- board text removed: "rx"
- board text removed: "tx"

Commit message: pushing workspace
Parts:
- C1, C2, C3, C4, C5, C6, C7: footprint Capacitor_SMD:C_0504_1310Metric_Pad0.83x1.28mm_HandSolder -> Capacitor_SMD:C_0805_2012Metric_Pad1.18x1.45mm_HandSolder
