File: PCB/MotorControl-2025-09-30_234331/MotorControl.kicad_pcb (KiCad board)
At the start: 2 copper layers, 117.9 x 76.4 mm, 15 parts, among them J1 Conn_01x03_Pin, J2 Conn_01x03_Pin, J3 Conn_01x03_Pin, J4 Conn_01x03_Pin, J5 Conn_01x05_Pin, J6 USB_C_Receptacle_USB2.0_14P, J7 Conn_01x03_Pin, U1 PCA9685PW, U2 NORA-W106-00B, U3 TC1262-33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

Commit message: Stuff
Routing:
- net 5V: track 254.3 -> 246.1 mm
- net TX: track 17.3 -> 22.1 mm
- net SWDIO: track 35.9 -> 31.3 mm
- net RX: track 21.3 -> 18.5 mm
- net NRST: track 45.4 -> 47.7 mm
- net SWSCLK: track 35.6 -> 34.0 mm
- net +3.3V: track 17.5 -> 18.2 mm
