File: PCB/MotorControl/MotorControl.kicad_pcb (KiCad board)
At the start: 2 copper layers, 117.9 x 76.4 mm, 28 parts, among them J1 Conn_01x03_Pin, J2 Conn_01x03_Pin, J3 Conn_01x03_Pin, J4 Conn_01x03_Pin, J5 Conn_01x05_Pin, J6 USB_C_Receptacle_USB2.0_14P, J7 Conn_01x03_Pin, J9 Conn_01x06_Socket, U1 PCA9685PW, U2 NORA-W106-00B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

Commit message: Boom
Parts:
- moved C3 0.38 mm to (101.0, 63.1)
Routing:
- net +3.3V: track 43.5 -> 34.9 mm, vias 8 -> 9
- net Net-(J7-Pin_3): track 44.7 -> 39.0 mm
- net GND: track 7.38 -> 2.70 mm
- net Motor1PWM: track 47.2 -> 43.8 mm
- net Net-(J2-Pin_3): track 31.4 -> 30.1 mm
- net Net-(J4-Pin_3): track 33.2 -> 32.2 mm
- net MotorControl_SCL: track 69.5 -> 68.7 mm
Changed lines of the file:
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@@
 	(footprint "Capacitor_SMD:C_0504_1310Metric_Pad0.83x1.28mm_HandSolder"
 		(layer "F.Cu")
-		(at 101.4297 63.0682 180)
+		(at 101.0458 63.0682 180)
 		(descr "Capacitor SMD 0504 (1310 Metric), square (rectangular) end terminal, IPC-7351 nominal with elongated pad for handsoldering. (Body size source: IPC-SM-782 page 76, https://www.pcb-3d.com/wordpress/wp-content/uploads/ipc-sm-782a_amendment_1_and_2.pdf), generated with kicad-footprint-generator")
 		(tags "capacitor handsolder")
@@
 	)
 	(segment
-		(start 126.1364 51.0286)
-		(end 128.7178 51.0286)
-		(width 0.2)
-		(layer "F.Cu")
-		(net 1)
-	)
-	(segment
 		(start 87.4834 100.4884)
 		(end 88.5834 100.4884)
@@
 	)
 	(segment
-		(start 103.8352 61.2902)
-		(end 102.0572 63.0682)
-		(width 0.2)
-		(layer "F.Cu")
-		(net 1)
-	)
-	(segment
 		(start 88.58 98.61)
 		(end 89.14 98.61)
@@
 	)
 	(segment
-		(start 102.7183 60.1479)
-		(end 102.7183 58.5474)
-		(width 0.2)
-		(layer "F.Cu")
-		(net 1)
-	)
-	(segment
 		(start 114.405 84.7886)
 		(end 116.4556 84.7886)
@@
 	)
 	(segment
-		(start 103.8606 61.2902)
-		(end 103.8352 61.2902)
-		(width 0.2)
-		(layer "F.Cu")
-		(net 1)
-	)
-	(segment
-		(start 126.0094 50.9016)
-		(end 126.1364 51.0286)
-		(width 0.2)
-		(layer "F.Cu")
-		(net 1)
-	)
-	(segment
 		(start 87.4834 101.5884)
 		(end 87.4834 100.4884)
@@
 	)
 	(segment
-		(start 103.8606 61.2902)
-		(end 102.7183 60.1479)
-		(width 0.2)
-		(layer "F.Cu")
-		(net 1)
-	)
-	(segment
 		(start 124.8056 90.3886)
 		(end 127.1932 90.3886)
@@
 	)
 	(via
-		(at 154.19 81.48)
+		(at 128.7178 51.0286)
 		(size 0.6)
 		(drill 0.3)
 		(layers "F.Cu" "B.Cu")
-		(free yes)
 		(net 1)
 	)
 	(via
-		(at 103.8606 61.2902)
+		(at 154.19 81.3792)
 		(size 0.6)
 		(drill 0.3)
@@
 	)
 	(via
-		(at 126.0094 50.9016)
+		(at 114.3508 84.7344)
 		(size 0.6)
 		(drill 0.3)
@@
 	)
 	(via
-		(at 114.3508 84.7344)
+		(at 127.3302 90.5256)
 		(size 0.6)
 		(drill 0.3)
@@
 	)
 	(via
-		(at 127.3302 90.5256)
+		(at 101.6733 63.0682)
+		(size 0.6)
+		(drill 0.3)
+		(layers "F.Cu" "B.Cu")
+		(net 1)
+	)
+	(via
+		(at 102.7183 58.5474)
 		(size 0.6)
 		(drill 0.3)
 		(layers "F.Cu" "B.Cu")
-		(free yes)
 		(net 1)
 	)
@@
 	)
 	(segment
-		(start 100.4183 58.5474)
-		(end 100.4183 62.6843)
-		(width 0.2)
-		(layer "F.Cu")
-		(net 2)
-	)
-	(segment
-		(start 100.4183 62.6843)
-		(end 100.8022 63.0682)
-		(width 0.2)
-		(layer "F.Cu")
-		(net 2)
-	)
-	(segment
 		(start 84.4414 70.939)
 		(end 83.0914 70.939)
@@
 	)
 	(segment
-		(start 177.62 53.3676)
-		(end 180.7464 50.2412)
+		(start 185.0228 46.5074)
+		(end 181.289 50.2412)
 		(width 0.2)
 		(layer "F.Cu")
@@
 	)
 	(segment
-		(start 166.6494 75.5396)
-		(end 166.6494 73.3806)
+		(start 177.62 53.3676)
+		(end 180.7464 50.2412)
 		(width 0.2)
 		(layer "F.Cu")
@@
 	(segment
 		(start 163.5352 75.5292)
-		(end 166.639 75.5292)
+		(end 164.5008 75.5292)
 		(width 0.2)
 		(layer "F.Cu")
@@
 	)
 	(segment
-		(start 181.1528 46.5074)
-		(end 181.0766 46.4312)
-		(width 0.2)
-		(layer "F.Cu")
-		(net 37)
-	)
-	(segment
-		(start 185.0228 46.5074)
-		(end 181.1528 46.5074)
-		(width 0.2)
-		(layer "F.Cu")
-		(net 37)
-	)
-	(segment
-		(start 180.7464 46.7614)
+		(start 181.289 50.2412)
 		(end 180.7464 50.2412)
 		(width 0.2)
@@
 	)
 	(segment
-		(start 181.0766 46.4312)
-		(end 180.7464 46.7614)
-		(width 0.2)
-		(layer "F.Cu")
-		(net 37)
-	)
-	(segment
-		(start 166.639 75.5292)
-		(end 166.6494 75.5396)
+		(start 164.5008 75.5292)
+		(end 166.6494 73.3806)
 		(width 0.2)
 		(layer "F.Cu")
@@
 	)
 	(segment
-		(start 167.9148 76.1792)
-		(end 167.9448 76.1492)
-		(width 0.2)
-		(layer "F.Cu")
-		(net 47)
-	)
-	(segment
 		(start 184.9974 61.7728)
 		(end 184.9974 66.2594)
@@
 	(segment
 		(start 163.5352 76.1792)
-		(end 167.9148 76.1792)
+		(end 165.7558 76.1792)
 		(width 0.2)
 		(layer "F.Cu")
@@
 	)
 	(segment
-		(start 167.9448 76.1492)
+		(start 165.7558 76.1792)
 		(end 167.9448 73.9902)
 		(width 0.2)
@@
 	)
 	(segment
-		(start 163.5352 77.4792)
-		(end 167.9794 77.4792)
-		(width 0.2)
-		(layer "F.Cu")
-		(net 49)
-	)
-	(segment
 		(start 167.9956 79.248)
 		(end 167.9956 79.3242)
@@
 	)
 	(segment
-		(start 168.021 77.5208)
-		(end 167.9956 77.5462)
+		(start 163.5352 77.4792)
+		(end 166.2268 77.4792)
 		(width 0.2)
 		(layer "F.Cu")
@@
 	)
 	(segment
-		(start 167.9956 77.5462)
-		(end 167.9956 79.248)
-		(width 0.2)
-		(layer "F.Cu")
-		(net 49)
-	)
-	(segment
-		(start 167.9794 77.4792)
-		(end 168.021 77.5208)
+		(start 185.099 94.7928)
+		(end 178.1048 94.7928)
 		(width 0.2)
 		(layer "F.Cu")
@@
 	)
 	(segment
-		(start 185.099 94.7928)
-		(end 178.1048 94.7928)
+		(start 166.2268 77.4792)
+		(end 167.9956 79.248)
 		(width 0.2)
 		(layer "F.Cu")
@@
 	)
 	(segment
-		(start 166.5212 78.1292)
-		(end 163.5352 78.1292)
-		(width 0.2)
-		(layer "F.Cu")
-		(net 50)
-	)
-	(segment
-		(start 185.0228 107.4674)
-		(end 177.0043 107.4674)
-		(width 0.2)
-		(layer "F.Cu")
-		(net 50)
-	)
-	(segment
-		(start 166.4716 80.4926)
-		(end 166.5224 80.4418)
-		(width 0.2)
-		(layer "F.Cu")
-		(net 50)
-	)
-	(segment
-		(start 166.4716 96.9347)
-		(end 166.4716 80.4926)
+		(start 171.75 85)
+		(end 171.75 94.1946)
 		(width 0.2)
 		(layer "F.Cu")
@@
 	)
 	(segment
-		(start 177.0043 107.4674)
-		(end 166.4716 96.9347)
+		(start 171.75 94.1946)
+		(end 185.0228 107.4674)
 		(width 0.2)
 		(layer "F.Cu")
@@
 	)
 	(segment
-		(start 166.5224 80.4418)
-		(end 166.5224 78.1304)
+		(start 164.8792 78.1292)
+		(end 171.75 85)
 		(width 0.2)
 		(layer "F.Cu")
@@
 	)
 	(segment
-		(start 166.5224 78.1304)
-		(end 166.5212 78.1292)
+		(start 163.5352 78.1292)
+		(end 164.8792 78.1292)
 		(width 0.2)
 		(layer "F.Cu")
@@
 	)
 	(segment
+		(start 132.7892 80.0792)
+		(end 157.8102 80.0792)
+		(width 0.2)
+		(layer "F.Cu")
+		(net 111)
+	)
+	(segment
 		(start 120.2306 83.4136)
 		(end 120.2306 79.0806)
@@
 	(segment
 		(start 131.34 78.63)
-		(end 131.34 80.0392)
-		(width 0.2)
-		(layer "F.Cu")
-		(net 111)
-	)
-	(segment
-		(start 157.8102 80.0792)
-		(end 131.38 80.0792)
-		(width 0.2)
-		(layer "F.Cu")
-		(net 111)
-	)
-	(segment
-		(start 131.34 80.0392)
-		(end 131.38 80.0792)
+		(end 132.7892 80.0792)
 		(width 0.2)
 		(layer "F.Cu")
