File: PCB/MotorControl/MotorControl.kicad_pcb (KiCad board)
At the start: 2 copper layers, 117.9 x 76.4 mm, 28 parts, among them J1 Conn_01x03_Pin, J2 Conn_01x03_Pin, J3 Conn_01x03_Pin, J4 Conn_01x03_Pin, J5 Conn_01x05_Pin, J6 USB_C_Receptacle_USB2.0_14P, J7 Conn_01x03_Pin, J9 Conn_01x06_Socket, U1 PCA9685PW, U2 NORA-W106-00B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

Commit message: wasd
Parts:
- added J10: Conn_01x01_Pin, Connector_PinHeader_2.54mm:PinHeader_1x01_P2.54mm_Vertical, F.Cu at (107.4, 83.3)
- added J8: Barrel_Jack, Connector_BarrelJack:BarrelJack_CUI_PJ-063AH_Horizontal, F.Cu at (155.1, 51.3)
- added R3: 270, Resistor_SMD:R_0805_2012Metric_Pad1.20x1.40mm_HandSolder, F.Cu at (103.4, 86.6)
Connections:
- U4 pad 31: GND -> Boot
Routing:
- net 5V: track 227.9 -> 9.38 mm
- net Boot: track 0.00 -> 18.6 mm, vias 0 -> 1
- net TX: track 33.7 -> 35.1 mm
- added copper zone on In1.Cu, net 5V
Other:
- outline, holes or cut-outs redrawn
- copper layers 2 -> 4
- board text added: "Boot"

Commit message: wasd
Routing:
- net +3.3V: track 34.9 -> 70.6 mm, vias 9 -> 7
- net 5V: track 9.38 -> 22.5 mm
- net MotorControl_SCL: track 68.7 -> 81.1 mm, vias 3 -> 2
- net GND: track 2.70 -> 0.00 mm
- net Boot: track 18.6 -> 18.7 mm, vias 1 -> 2
- added copper zone on B.Cu, net 5V
- removed copper zone on In1.Cu, net 5V
Other:
- copper layers 4 -> 2

Commit message: final boards
Parts:
- J6: value USB_C_Receptacle_USB2.0_14P -> Conn_01x02_Socket; footprint Connector_USB:USB_C_Receptacle_GCT_USB4085 -> Connector_PinSocket_2.54mm:PinSocket_1x02_P2.54mm_Horizontal
- J8: footprint Connector_BarrelJack:BarrelJack_CUI_PJ-063AH_Horizontal -> Connector_BarrelJack:BarrelJack_Wuerth_694106106102_2.0x5.5mm
- moved J6 34.8 mm to (111.1, 48.6)
- moved J8 32.7 mm to (122.5, 48.7)
- moved TP2 29.4 mm to (149.1, 46.7)
- moved J2 28.6 mm to (156.4, 56.9)
- moved J1 28.6 mm to (156.4, 41.6)
- moved J3 28.6 mm to (156.4, 74.6)
- moved J4 28.6 mm to (156.5, 89.9)
- moved J7 28.6 mm to (156.4, 102.6)
- moved U1 17.1 mm to (143.6, 77.6)
- moved R4 11.5 mm to (121.6, 59.2)
- moved D3 11.5 mm to (129.7, 59.2)
- moved J5 4.36 mm to (146.8, 85.9)
- moved C7 4.19 mm to (89.0, 96.0)
- moved C6 3.64 mm to (92.0, 96.0)
- moved C5 2.80 mm to (86.5, 96.0)
Connections:
- R2 pad 1: GND -> +3.3V
- U2 pad L1: unconnected-(U2-EAGP-PadL1)_2 -> GND
- U2 pad L9: unconnected-(U2-EAGP-PadL1)_3 -> GND
- U2 pad M1: unconnected-(U2-EAGP-PadL1) -> GND
- U2 pad M2: unconnected-(U2-EAGP-PadL1)_1 -> GND
- U2 pad M8: unconnected-(U2-EAGP-PadL1)_5 -> GND
- U2 pad M9: unconnected-(U2-EAGP-PadL1)_4 -> GND
Routing:
- net MotorControl_SCL: track 81.1 -> 45.0 mm
- net Net-(U1-SDA): track 41.3 -> 24.4 mm
- net +3.3V: track 70.6 -> 57.2 mm, vias 7 -> 12
- net Net-(J3-Pin_3): track 22.9 -> 11.1 mm, vias 2 -> 1
- net Net-(J2-Pin_3): track 30.1 -> 20.1 mm, vias 2 -> 1
- net Net-(J4-Pin_3): track 32.2 -> 22.9 mm, vias 2 -> 1
- net 5V: track 22.5 -> 15.1 mm, vias 0 -> 9
- net Switch1: track 49.1 -> 43.7 mm
- net Net-(J7-Pin_3): track 39.0 -> 34.0 mm
- net SWSCLK: track 28.9 -> 24.6 mm
- net SWDIO: track 29.7 -> 25.3 mm
- net NRST: track 46.3 -> 42.7 mm
- net Motor1PWM: track 43.8 -> 41.3 mm, vias 2 -> 1
- net Switch2: track 49.1 -> 47.3 mm
Other:
- board size 117.9 x 76.4 mm -> 90.1 x 94.1 mm
- board text added: "5v"

Commit message: pushing workspace
Parts:
- C1, C2, C3, C4, C5, C6, C7: footprint Capacitor_SMD:C_0504_1310Metric_Pad0.83x1.28mm_HandSolder -> Capacitor_SMD:C_0805_2012Metric_Pad1.18x1.45mm_HandSolder
Routing:
- net NRST: track 42.7 -> 42.2 mm
Other:
- board size 90.1 x 94.1 mm -> 90.1 x 94.5 mm
