File: PCB/RemoteControl_HighPowerAmp/RemoteControl.kicad_sch (KiCad schematic)
At the start: 58 parts, among them J1 Barrel_Jack, J10 Conn_01x01_Pin, J11 Conn_01x02_Socket, J3 Conn_01x05_Pin, J4 Conn_01x02_Socket, J5 Conn_01x06_Socket, J6 Conn_01x02_Socket, J7 Conn_01x02_Socket, J8 Conn_01x02_Socket, J9 Conn_01x02_Socket, U1 STM32L031K6Tx, U2 TC1262-33, U3 NORA-W106-00B, U4 LM358APE4, U5 LM358APE4, U6 LM358APE4, U7 LM358APE4, U8 LM358APE4

Commit message: final boards
Parts:
- removed U4, U5, U6, U7, U8: LM358APE4, lm358:P8, symbol 2025-10-16_17-58-12:LM358APE4
- added U10, U11, U12, U13, U4, U5, U6, U7, U8, U9: TL071CP, TL071CP:DIP794W45P254L959H508Q8, symbol TL071CP:TL071CP
- J1: footprint Connector_BarrelJack:BarrelJack_Wuerth_694106106102_2.0x5.5mm -> Connector_BarrelJack:BarrelJack_CUI_PJ-063AH_Horizontal
Connections:
- net +3.3V: no longer R7.1
- net +5V: now also U10.7 (VCC+), U11.7 (VCC+), U12.7 (VCC+), U13.7 (VCC+), U4.7 (VCC+), U5.7 (VCC+), U6.7 (VCC+), U7.7 (VCC+), U8.7 (VCC+), U9.7 (VCC+)
- net Finger1: now also U11.2 (IN-), U11.6 (OUT)
- net Finger2: now also U9.2 (IN-), U9.6 (OUT)
- net Finger3: now also U13.2 (IN-), U13.6 (OUT)
- net Finger4: now also U4.2 (IN-), U4.6 (OUT)
- net Finger5: now also U7.2 (IN-), U7.6 (OUT)
- net GND: now also R7.1, U10.1 (OFFSET_N1), U10.4 (VCC-), U10.5 (OFFSET_N2), U11.1 (OFFSET_N1), U11.4 (VCC-), U11.5 (OFFSET_N2), U12.1 (OFFSET_N1), U12.4 (VCC-), U12.5 (OFFSET_N2), U13.1 (OFFSET_N1), U13.4 (VCC-), U13.5 (OFFSET_N2), U4.1 (OFFSET_N1), U4.4 (VCC-), U4.5 (OFFSET_N2), U5.1 (OFFSET_N1), U5.4 (VCC-), U5.5 (OFFSET_N2), U6.1 (OFFSET_N1), U6.4 (VCC-), U6.5 (OFFSET_N2), U7.1 (OFFSET_N1), U7.4 (VCC-), U7.5 (OFFSET_N2), U8.1 (OFFSET_N1), U8.4 (VCC-), U8.5 (OFFSET_N2), U9.1 (OFFSET_N1), U9.4 (VCC-), U9.5 (OFFSET_N2); no longer U3.L1 (EAGP), U3.L9 (EAGP), U3.M1 (EAGP), U3.M2 (EAGP), U3.M8 (EAGP), U3.M9 (EAGP)
- net Sensor1: now also U12.3 (IN+)
- net Sensor2: now also U5.3 (IN+)
- net Sensor3: now also U6.3 (IN+)
- net Sensor4: now also U8.3 (IN+)
- net Sensor5: now also U10.3 (IN+)
- net at R13.1: now also U4.3 (IN+), U5.6 (OUT)
- net at R12.2, R13.2: now also U5.2 (IN-)
- net at R18.2, R19.1: now also U10.2 (IN-)
- net at R19.2: now also U10.6 (OUT), U11.3 (IN+)
- net at R17.2: now also U8.6 (OUT), U9.3 (IN+)
- net at R16.2, R17.1: now also U8.2 (IN-)
- net at R14.1: now also U6.6 (OUT), U7.3 (IN+)
- net at R14.2, R15.2: now also U6.2 (IN-)
- net at R11.1: now also U12.6 (OUT), U13.3 (IN+)
- net at R10.2, R11.2: now also U12.2 (IN-)
- new net: U3.L1 (EAGP), U3.L9 (EAGP), U3.M1 (EAGP), U3.M2 (EAGP), U3.M8 (EAGP), U3.M9 (EAGP)
- no-connect marks 47 -> 48
Other:
- moved on the sheet: R10, R11
